File: test.kicad_pcb (KiCad board)
At the start: 2 copper layers, 79 parts, among them Q1 T2N7002AK, Q2 T2N7002AK, SW1 SW_Push, U1 ESP32-S3-WROOM-1, U2 LD1117S33TR_SOT223, U3 AT45DB161D-SU, Y1 Crystal

Commit message: schematic almost complete
Parts:
- added U3: SN75176AD, Package_SO:SOIC-8_3.9x4.9mm_P1.27mm, F.Cu at (244.3, 28.7)
- added U4: LM321, Package_TO_SOT_SMD:SOT-23-5, F.Cu at (242.6, 34.3)
- added U5: LM321, Package_TO_SOT_SMD:SOT-23-5, F.Cu at (242.6, 38.9)
- added aco1: PC817, Package_DIP:DIP-4_W7.62mm_SMDSocket_SmallPads, F.Cu at (205.8, 22.0)
- added aco2: PC817, Package_DIP:DIP-4_W7.62mm_SMDSocket_SmallPads, F.Cu at (205.8, 28.8)
- added bridge1: MB1S, Diode_SMD:Diode_Bridge_OnSemi_SDIP-4L, F.Cu at (244.8, 57.3)
- added bridge2: MB1S, Diode_SMD:Diode_Bridge_OnSemi_SDIP-4L, F.Cu at (244.8, 67.1)
- added c3: 100nF, Capacitor_SMD:C_0805_2012Metric_Pad1.18x1.45mm_HandSolder, F.Cu at (247.6, 33.4)
- added cf1: 100nF, Capacitor_SMD:C_0805_2012Metric_Pad1.18x1.45mm_HandSolder, F.Cu at (247.6, 36.4)
- added cr2: C_Polarized, Capacitor_THT:CP_Axial_L30.0mm_D10.0mm_P35.00mm_Horizontal, F.Cu at (201.9, 58.1)
- added cr3: C_Polarized, Capacitor_THT:CP_Axial_L30.0mm_D10.0mm_P35.00mm_Horizontal, F.Cu at (201.9, 69.7)
- added di1: 1N4148W, Diode_SMD:D_SOD-123, F.Cu at (181.7, 84.3)
- added di2: 1N4148W, Diode_SMD:D_SOD-123, F.Cu at (181.7, 87.7)
- added di3: 1N4148W, Diode_SMD:D_SOD-123, F.Cu at (181.7, 91.0)
- added di4: 1N4148W, Diode_SMD:D_SOD-123, F.Cu at (181.7, 94.4)
- added di5: 1N4148W, Diode_SMD:D_SOD-123, F.Cu at (187.5, 84.3)
- added di6: 1N4148W, Diode_SMD:D_SOD-123, F.Cu at (187.5, 87.7)
- added di7: 1N4148W, Diode_SMD:D_SOD-123, F.Cu at (187.5, 91.0)
- added di8: 1N4148W, Diode_SMD:D_SOD-123, F.Cu at (187.5, 94.4)
- added dr1: 1N4148W, Diode_SMD:D_SOD-123, F.Cu at (193.3, 84.3)
- added dr2: 1N4148W, Diode_SMD:D_SOD-123, F.Cu at (193.3, 87.7)
- added dr3: 1N4148W, Diode_SMD:D_SOD-123, F.Cu at (193.3, 91.0)
- added dr4: 1N4148W, Diode_SMD:D_SOD-123, F.Cu at (193.3, 94.4)
- added dz1: D_Zener, Diode_SMD:D_MiniMELF_Handsoldering, F.Cu at (245.3, 20.3)
- added dz2: D_Zener, Diode_SMD:D_MiniMELF_Handsoldering, F.Cu at (245.3, 23.6)
- added in1: PC817, Package_DIP:DIP-4_W7.62mm_SMDSocket_SmallPads, F.Cu at (205.8, 35.5)
- added in2: PC817, Package_DIP:DIP-4_W7.62mm_SMDSocket_SmallPads, F.Cu at (205.8, 42.2)
- added in3: PC817, Package_DIP:DIP-4_W7.62mm_SMDSocket_SmallPads, F.Cu at (205.8, 49.0)
- added in4: PC817, Package_DIP:DIP-4_W7.62mm_SMDSocket_SmallPads, F.Cu at (217.5, 22.0)
- added in5: PC817, Package_DIP:DIP-4_W7.62mm_SMDSocket_SmallPads, F.Cu at (217.5, 28.8)
- added in6: PC817, Package_DIP:DIP-4_W7.62mm_SMDSocket_SmallPads, F.Cu at (217.5, 35.5)
- added in7: PC817, Package_DIP:DIP-4_W7.62mm_SMDSocket_SmallPads, F.Cu at (217.5, 42.2)
- added in8: PC817, Package_DIP:DIP-4_W7.62mm_SMDSocket_SmallPads, F.Cu at (217.5, 49.0)
- added out1: PC817, Package_DIP:DIP-4_W7.62mm_SMDSocket_SmallPads, F.Cu at (229.3, 22.0)
- added out2: PC817, Package_DIP:DIP-4_W7.62mm_SMDSocket_SmallPads, F.Cu at (229.3, 28.8)
- added out3: PC817, Package_DIP:DIP-4_W7.62mm_SMDSocket_SmallPads, F.Cu at (229.3, 35.5)
- added out4: PC817, Package_DIP:DIP-4_W7.62mm_SMDSocket_SmallPads, F.Cu at (229.3, 42.2)
- added qm1: PMBT2222A, Package_TO_SOT_SMD:SOT-23, F.Cu at (237.6, 21.0)
- added qr1: PMBT2222A, Package_TO_SOT_SMD:SOT-23, F.Cu at (237.6, 25.6)
- added qr2: PMBT2222A, Package_TO_SOT_SMD:SOT-23, F.Cu at (237.6, 30.3)
- added qr3: PMBT2222A, Package_TO_SOT_SMD:SOT-23, F.Cu at (237.6, 34.9)
- added qr4: PMBT2222A, Package_TO_SOT_SMD:SOT-23, F.Cu at (237.6, 39.5)
- added r1: 7.5K, Resistor_SMD:R_1206_3216Metric_Pad1.30x1.75mm_HandSolder, F.Cu at (181.7, 71.1)
- added r10: 2.8K, Resistor_SMD:R_1206_3216Metric_Pad1.30x1.75mm_HandSolder, F.Cu at (187.7, 74.4)
- added r11: 7.5K, Resistor_SMD:R_1206_3216Metric_Pad1.30x1.75mm_HandSolder, F.Cu at (187.7, 77.7)
- added r12: 7.5K, Resistor_SMD:R_1206_3216Metric_Pad1.30x1.75mm_HandSolder, F.Cu at (187.7, 81.0)
- added r13: 680, Resistor_SMD:R_0805_2012Metric_Pad1.20x1.40mm_HandSolder, F.Cu at (202.3, 88.8)
- added r14: 680, Resistor_SMD:R_0805_2012Metric_Pad1.20x1.40mm_HandSolder, F.Cu at (202.3, 91.7)
- added r15: 680, Resistor_SMD:R_0805_2012Metric_Pad1.20x1.40mm_HandSolder, F.Cu at (202.3, 94.7)
- added r16: 680, Resistor_SMD:R_0805_2012Metric_Pad1.20x1.40mm_HandSolder, F.Cu at (207.0, 77.0)
- added r17: 1K, Resistor_SMD:R_0805_2012Metric_Pad1.20x1.40mm_HandSolder, F.Cu at (207.0, 79.9)
- added r18: 1K, Resistor_SMD:R_0805_2012Metric_Pad1.20x1.40mm_HandSolder, F.Cu at (207.0, 82.8)
- added r19: 560, Resistor_SMD:R_0805_2012Metric_Pad1.20x1.40mm_HandSolder, F.Cu at (207.0, 85.8)
- added r2: 7.5K, Resistor_SMD:R_1206_3216Metric_Pad1.30x1.75mm_HandSolder, F.Cu at (181.7, 74.4)
- added r20: 560, Resistor_SMD:R_0805_2012Metric_Pad1.20x1.40mm_HandSolder, F.Cu at (207.0, 88.8)
- added r21: 100K, Resistor_SMD:R_0805_2012Metric_Pad1.20x1.40mm_HandSolder, F.Cu at (207.0, 91.7)
- added r22: 100K, Resistor_SMD:R_0805_2012Metric_Pad1.20x1.40mm_HandSolder, F.Cu at (207.0, 94.7)
- added r23: 10K, Resistor_SMD:R_0805_2012Metric_Pad1.20x1.40mm_HandSolder, F.Cu at (211.8, 77.0)
- added r24: 10K, Resistor_SMD:R_0805_2012Metric_Pad1.20x1.40mm_HandSolder, F.Cu at (211.8, 79.9)
- added r25: 120, Resistor_SMD:R_0805_2012Metric_Pad1.20x1.40mm_HandSolder, F.Cu at (211.8, 82.8)
- added r26: 10K, Resistor_SMD:R_0805_2012Metric_Pad1.20x1.40mm_HandSolder, F.Cu at (211.8, 85.8)
- added r27: 10K, Resistor_SMD:R_0805_2012Metric_Pad1.20x1.40mm_HandSolder, F.Cu at (211.8, 88.8)
- added r28: 2.7K, Resistor_SMD:R_1206_3216Metric_Pad1.30x1.75mm_HandSolder, F.Cu at (193.6, 71.1)
- added r29: 2.7K, Resistor_SMD:R_1206_3216Metric_Pad1.30x1.75mm_HandSolder, F.Cu at (193.6, 74.4)
- added r3: 7.5K, Resistor_SMD:R_1206_3216Metric_Pad1.30x1.75mm_HandSolder, F.Cu at (181.7, 77.7)
- added r30: 3.3K, Resistor_SMD:R_0805_2012Metric_Pad1.20x1.40mm_HandSolder, F.Cu at (211.8, 91.7)
- added r31: 3.3K, Resistor_SMD:R_0805_2012Metric_Pad1.20x1.40mm_HandSolder, F.Cu at (211.8, 94.7)
- added r32: 2.7K, Resistor_SMD:R_1206_3216Metric_Pad1.30x1.75mm_HandSolder, F.Cu at (193.6, 77.7)
- added r33: 2.7K, Resistor_SMD:R_1206_3216Metric_Pad1.30x1.75mm_HandSolder, F.Cu at (193.6, 81.0)
- added r34: 3.3K, Resistor_SMD:R_0805_2012Metric_Pad1.20x1.40mm_HandSolder, F.Cu at (216.5, 77.0)
- added r35: 3.3K, Resistor_SMD:R_0805_2012Metric_Pad1.20x1.40mm_HandSolder, F.Cu at (216.5, 79.9)
- added r4: 7.5K, Resistor_SMD:R_1206_3216Metric_Pad1.30x1.75mm_HandSolder, F.Cu at (181.7, 81.0)
- added r5: 680, Resistor_SMD:R_0805_2012Metric_Pad1.20x1.40mm_HandSolder, F.Cu at (202.3, 77.0)
- added r6: 680, Resistor_SMD:R_0805_2012Metric_Pad1.20x1.40mm_HandSolder, F.Cu at (202.3, 79.9)
- added r7: 680, Resistor_SMD:R_0805_2012Metric_Pad1.20x1.40mm_HandSolder, F.Cu at (202.3, 82.8)
- added r8: 680, Resistor_SMD:R_0805_2012Metric_Pad1.20x1.40mm_HandSolder, F.Cu at (202.3, 85.8)
- added r9: 2.5K, Resistor_SMD:R_1206_3216Metric_Pad1.30x1.75mm_HandSolder, F.Cu at (187.7, 71.1)
- added ra1: 100K, Resistor_SMD:R_0805_2012Metric_Pad1.20x1.40mm_HandSolder, F.Cu at (216.5, 82.8)
- added ra2: 100K, Resistor_SMD:R_0805_2012Metric_Pad1.20x1.40mm_HandSolder, F.Cu at (216.5, 85.8)
- added ra3: 33K, Resistor_SMD:R_0805_2012Metric_Pad1.20x1.40mm_HandSolder, F.Cu at (216.5, 88.8)
- added ra4: 33K, Resistor_SMD:R_0805_2012Metric_Pad1.20x1.40mm_HandSolder, F.Cu at (216.5, 91.7)
- added ra5: 68, Resistor_SMD:R_0805_2012Metric_Pad1.20x1.40mm_HandSolder, F.Cu at (216.5, 94.7)
- added ra6: 68, Resistor_SMD:R_0805_2012Metric_Pad1.20x1.40mm_HandSolder, F.Cu at (221.3, 77.0)
- added rb1: 100K, Resistor_THT:R_Axial_DIN0414_L11.9mm_D4.5mm_P20.32mm_Horizontal, F.Cu at (225.6, 78.5)
- added rb2: 100K, Resistor_THT:R_Axial_DIN0414_L11.9mm_D4.5mm_P20.32mm_Horizontal, F.Cu at (225.6, 84.5)
- added relay2: SANYOU_SRD_Form_C, Relay_THT:Relay_SPDT_SANYOU_SRD_Series_Form_C, F.Cu at (180.8, 27.1)
- added relay3: SANYOU_SRD_Form_C, Relay_THT:Relay_SPDT_SANYOU_SRD_Series_Form_C, F.Cu at (180.8, 44.0)
- added relay4: SANYOU_SRD_Form_C, Relay_THT:Relay_SPDT_SANYOU_SRD_Series_Form_C, F.Cu at (180.8, 61.0)
- added rf1: 100K, Resistor_SMD:R_0805_2012Metric_Pad1.20x1.40mm_HandSolder, F.Cu at (221.3, 79.9)
- added rf2: 100K, Resistor_SMD:R_0805_2012Metric_Pad1.20x1.40mm_HandSolder, F.Cu at (221.3, 82.8)
- added rlb1: 1K, Resistor_SMD:R_0805_2012Metric_Pad1.20x1.40mm_HandSolder, F.Cu at (221.3, 85.8)
- added rlb2: 1K, Resistor_SMD:R_0805_2012Metric_Pad1.20x1.40mm_HandSolder, F.Cu at (221.3, 88.8)
- added rlb3: 1K, Resistor_SMD:R_0805_2012Metric_Pad1.20x1.40mm_HandSolder, F.Cu at (221.3, 91.7)
- added rlb4: 1K, Resistor_SMD:R_0805_2012Metric_Pad1.20x1.40mm_HandSolder, F.Cu at (221.3, 94.7)
- moved opt14 13.9 mm to (65.5, 112.1)
- moved ebt1 10.0 mm to (98.7, 111.3)
- moved cch2 2.49 mm to (74.2, 92.0)
- renumbered U3 to flash1, rel1 to relay1
Connections:
- flash1 pad 1: unconnected-(U3-SI-Pad1) -> /SI
- flash1 pad 2: unconnected-(U3-SCK-Pad2) -> /SCK
- flash1 pad 3: unconnected-(U3-~{RESET}-Pad3) -> /FRES
- flash1 pad 4: unconnected-(U3-~{CS}-Pad4) -> /CS
- flash1 pad 5: unconnected-(U3-~{WP}-Pad5) -> Net-(flash1-~{WP})
- flash1 pad 6: unconnected-(U3-VCC-Pad6) -> /+3.3V
- flash1 pad 7: unconnected-(U3-GND-Pad7) -> GND
- flash1 pad 8: unconnected-(U3-SO-Pad8) -> /SO
- relay1 pad 2: unconnected-(rel1-Pad2) -> Net-(dr1-A)
- relay1 pad 5: unconnected-(rel1-Pad5) -> /+5V

Commit message: schematic complete
Parts:
- removed L0: L_Ferrite, Inductor_SMD:L_0805_2012Metric_Pad1.05x1.20mm_HandSolder
- removed Y1: Crystal, Crystal:Crystal_SMD_HC49-SD
- removed di1, di7: 1N4148W, Diode_SMD:D_SOD-123
- removed in1, in2, in5, in7, opt1, opt10, opt11, opt12, opt13, opt14, opt15, opt16, opt2, opt3, opt4, opt5, opt6, opt7, opt8, opt9: PC817, Package_DIP:DIP-4_W7.62mm_SMDSocket_SmallPads
- removed r11: 7.5K, Resistor_SMD:R_1206_3216Metric_Pad1.30x1.75mm_HandSolder
- removed r13, r15, r6: 680, Resistor_SMD:R_0805_2012Metric_Pad1.20x1.40mm_HandSolder
- removed the rb1 at (225.6, 78.5)
- removed rel2, rel3, rel4: SANYOU_SRD_Form_C, Relay_THT:Relay_SPDT_SANYOU_SRD_Series_Form_C
- added HS1: 6N137, Package_DIP:DIP-8_W7.62mm, F.Cu at (100.4, 16.2)
- added HS2: 6N137, Package_DIP:DIP-8_W7.62mm, F.Cu at (111.3, 16.2)
- added L1: L_Ferrite, Inductor_SMD:L_0805_2012Metric_Pad1.05x1.20mm_HandSolder, F.Cu at (117.9, 110.2)
- added OLED1: Conn_01x04_Pin, Connector_Molex:Molex_KK-254_AE-6410-04A_1x04_P2.54mm_Vertical, F.Cu at (-49.5, 75.2)
- added Sensor1: Conn_01x04_Pin, Connector_Molex:Molex_KK-254_AE-6410-04A_1x04_P2.54mm_Vertical, F.Cu at (-49.5, 83.1)
- added c4: 100nF, Capacitor_SMD:C_0805_2012Metric_Pad1.18x1.45mm_HandSolder, F.Cu at (91.7, 67.0)
- added c5: 100nF, Capacitor_SMD:C_0805_2012Metric_Pad1.18x1.45mm_HandSolder, F.Cu at (91.7, 70.0)
- added cm6: 100nF, Capacitor_SMD:C_0805_2012Metric_Pad1.18x1.45mm_HandSolder, F.Cu at (101.3, 73.0)
- added cm7: 100nF, Capacitor_SMD:C_0805_2012Metric_Pad1.18x1.45mm_HandSolder, F.Cu at (101.3, 76.0)
- added i2c1: 100K, Resistor_SMD:R_0805_2012Metric_Pad1.20x1.40mm_HandSolder, F.Cu at (88.0, 99.8)
- added i2c2: 100K, Resistor_SMD:R_0805_2012Metric_Pad1.20x1.40mm_HandSolder, F.Cu at (88.0, 102.7)
- added jadc1: 0, Resistor_SMD:R_0805_2012Metric_Pad1.20x1.40mm_HandSolder, F.Cu at (88.0, 105.7)
- added jadc2: 0, Resistor_SMD:R_0805_2012Metric_Pad1.20x1.40mm_HandSolder, F.Cu at (88.0, 108.6)
- added rb1: 100K, Resistor_THT:R_Axial_DIN0414_L11.9mm_D4.5mm_P20.32mm_Horizontal, F.Cu at (150.9, 117.7)
- added rb1: 100K, Resistor_THT:R_Axial_DIN0414_L11.9mm_D4.5mm_P20.32mm_Horizontal, F.Cu at (76.5, 17.2)
- cr2, cr3: footprint Capacitor_THT:CP_Axial_L30.0mm_D10.0mm_P35.00mm_Horizontal -> Capacitor_THT:CP_Radial_D22.0mm_P10.00mm_SnapIn
- r1: value 7.5K -> 680; footprint Resistor_SMD:R_1206_3216Metric_Pad1.30x1.75mm_HandSolder -> Resistor_SMD:R_0805_2012Metric_Pad1.20x1.40mm_HandSolder
- r2: value 7.5K -> 2.2K
- r9: value 2.5K -> 560
- ra1, ra2: value 100K -> 68K
- moved out1 290.1 mm to (-57.6, 64.9)
- moved out2 290.1 mm to (-57.6, 71.7)
- moved out3 290.1 mm to (-57.6, 78.4)
- moved out4 290.1 mm to (-57.6, 85.2)
- moved in4 276.1 mm to (-57.6, 44.7)
- moved in6 275.6 mm to (-57.6, 51.4)
- moved in8 275.3 mm to (-57.6, 58.2)
- moved in3 263.7 mm to (-57.6, 37.9)
- moved aco1 263.5 mm to (-57.6, 24.4)
- moved aco2 263.5 mm to (-57.6, 31.2)
- moved U3 191.1 mm to (56.1, 61.9)
- moved CH340 170.1 mm to (20.2, 54.0), turned to -90 degrees
- moved rb2 161.2 mm to (76.5, 23.2)
- moved c3 158.9 mm to (91.7, 63.9)
- moved cf1 154.2 mm to (96.5, 67.0)
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Connections:
- net /ADC1 renamed Net-(dz1-K)
- net /FRES renamed Net-(flash1-~{RESET})
- net Net-(aco1-Pad4) renamed /D220_IN1
- net Net-(aco2-Pad4) renamed /D220_IN2
- net Net-(in3-Pad4) renamed /D24_IN4
- net Net-(in4-Pad4) renamed /D24_IN1
- net Net-(in6-Pad4) renamed /D05_IN1
- net Net-(in8-Pad4) renamed /D24_IN3
- U2 pad 1: unconnected-(U2-GND-Pad1) -> GND
- cr2 pad 1: Net-(bridge1-+) -> Net-(cr2-Pad1)
- cr2 pad 2: Net-(bridge1--) -> Net-(bridge2--)
- cr3 pad 1: Net-(bridge2-+) -> Net-(cr3-Pad1)
- cr3 pad 2: Net-(bridge2--) -> Net-(bridge1--)
- mcu1 pad 12: unconnected-(mcu1-PA2-Pad12) -> /CHTXD
- mcu1 pad 13: unconnected-(mcu1-PA3-Pad13) -> /CHRXD
- mcu1 pad 14: unconnected-(mcu1-PA4-Pad14) -> /AIN1
- mcu1 pad 15: unconnected-(mcu1-PA5-Pad15) -> /AIN2
- mcu1 pad 25: unconnected-(mcu1-PB12-Pad25) -> /CS
- mcu1 pad 26: unconnected-(mcu1-PB13-Pad26) -> /SCK
- mcu1 pad 27: unconnected-(mcu1-PB14-Pad27) -> /SO
- mcu1 pad 28: unconnected-(mcu1-PB15-Pad28) -> /SI
- mcu1 pad 30: unconnected-(mcu1-PA9-Pad30) -> /UART1_TX
- mcu1 pad 31: unconnected-(mcu1-PA10-Pad31) -> /UART1_RX
- mcu1 pad 39: /SWO -> unconnected-(mcu1-PB3-Pad39)
- mcu1 pad 42: unconnected-(mcu1-PB6-Pad42) -> /I2C_SCL
- mcu1 pad 43: unconnected-(mcu1-PB7-Pad43) -> /I2C_SDA
- out2 pad 3: /DO3 -> /DO2
- out3 pad 3: /DO2 -> /DO3
- prg1 pad 5: /SWO -> /+3.3V
- r1 pad 1: /DI1 -> /D05_IN2
- r1 pad 2: Net-(di1-K) -> /+5V
- r17 pad 2: Net-(r17-Pad2) -> Net-(cr3-Pad1)
- r18 pad 2: Net-(r18-Pad2) -> Net-(cr2-Pad1)
- r19 pad 2: Net-(r17-Pad2) -> Net-(cr3-Pad1)
- r20 pad 2: Net-(r18-Pad2) -> Net-(cr2-Pad1)
- r29 pad 1: /MDO1 -> /MDO2
- r32 pad 1: /MDO1 -> /MDO3
- r33 pad 1: /MDO1 -> /MDO4
- r5 pad 1: Net-(in1-Pad4) -> /D24_IN2
- r5 pad 2: /+3.3V -> /+5V
- rb2 pad 2: Net-(r18-Pad2) -> Net-(cr2-Pad1)
- relay1 pad 1: unconnected-(relay1-Pad1) -> /RELOUT12
- relay1 pad 3: unconnected-(relay1-Pad3) -> /RELOUT11
- relay2 pad 1: unconnected-(relay2-Pad1) -> /RELOUT32
- relay2 pad 3: unconnected-(relay2-Pad3) -> /RELOUT31
- relay3 pad 1: unconnected-(relay3-Pad1) -> /RELOUT42
- relay3 pad 3: unconnected-(relay3-Pad3) -> /RELOUT41
- relay4 pad 1: unconnected-(relay4-Pad1) -> /RELOUT22
- relay4 pad 3: unconnected-(relay4-Pad3) -> /RELOUT21

Commit message: finished power and esp32 in pcb
Parts:
- removed ESP_GPIO1: Conn_02x11_Odd_Even, Connector_PinHeader_2.00mm:PinHeader_2x11_P2.00mm_Vertical
- removed the rb1 at (150.9, 117.7)
- removed the rb1 at (76.5, 17.2)
- added 220in1: Screw_Terminal_01x03, TerminalBlock:TerminalBlock_Altech_AK300-3_P5.00mm, F.Cu at (97.2, 89.7)
- added AIN1: Conn_01x03_Pin, Connector_Molex:Molex_KK-254_AE-6410-03A_1x03_P2.54mm_Vertical, F.Cu at (113.9, 51.3)
- added DDO1: Conn_01x08_Socket, Connector_Molex:Molex_KK-254_AE-6410-08A_1x08_P2.54mm_Vertical, F.Cu at (109.4, 17.3)
- added MODBUS1: Screw_Terminal_01x03, TerminalBlock:TerminalBlock_Altech_AK300-3_P5.00mm, F.Cu at (97.2, 103.7)
- added acin1: Screw_Terminal_01x02, TerminalBlock_MetzConnect:TerminalBlock_MetzConnect_Type011_RT05502HBWC_1x02_P5.00mm_Horizontal, F.Cu at (155.6, 38.4)
- added c6: 100nF, Capacitor_SMD:C_0805_2012Metric_Pad1.18x1.45mm_HandSolder, F.Cu at (48.3, 119.2)
- added c7: 100nF, Capacitor_SMD:C_0805_2012Metric_Pad1.18x1.45mm_HandSolder, F.Cu at (53.1, 104.2)
- added din1: Conn_01x07_Pin, Connector_Molex:Molex_KK-254_AE-6410-07A_1x07_P2.54mm_Vertical, F.Cu at (115.0, 75.2)
- added espio1: Conn_02x11_Odd_Even, Connector_PinHeader_2.00mm:PinHeader_2x11_P2.00mm_Vertical, F.Cu at (235.5, 20.3)
- added iso1: ADuM1201BR, Package_SO:SOIC-8_3.9x4.9mm_P1.27mm, F.Cu at (121.2, 125.6)
- added iso5: Conn_01x04_Pin, Connector_Molex:Molex_KK-254_AE-6410-04A_1x04_P2.54mm_Vertical, F.Cu at (64.3, 45.1)
- added rb1: 100K, Resistor_THT:R_Axial_DIN0414_L11.9mm_D4.5mm_P20.32mm_Horizontal, F.Cu at (64.0, 16.4)
- added relayout1: Conn_01x09_Pin, Connector_Molex:Molex_KK-254_AE-6410-09A_1x09_P2.54mm_Vertical, F.Cu at (99.6, 43.5)
- added rsj0: 0, Resistor_SMD:R_0805_2012Metric_Pad1.20x1.40mm_HandSolder, F.Cu at (91.5, 96.0)
- added rsj1: 0, Resistor_SMD:R_0805_2012Metric_Pad1.20x1.40mm_HandSolder, F.Cu at (91.5, 98.9)
- added rsjg1: 0, Resistor_SMD:R_0805_2012Metric_Pad1.20x1.40mm_HandSolder, F.Cu at (91.5, 101.9)
- C1: value 100nF -> C_Polarized; footprint Capacitor_SMD:C_0805_2012Metric_Pad1.18x1.45mm_HandSolder -> Capacitor_THT:CP_Radial_D4.0mm_P1.50mm
- C2: value 10uF -> C_Polarized; footprint Capacitor_SMD:C_0805_2012Metric_Pad1.18x1.45mm_HandSolder -> Capacitor_THT:CP_Radial_D4.0mm_P1.50mm
- U2: moved to B.Cu
- moved chusb1 269.0 mm to (279.7, -22.1), turned to 180 degrees
- moved CH340 265.0 mm to (276.7, -12.8), turned to 90 degrees
- moved U1 211.8 mm to (245.6, -0.92)
- moved cch1 207.2 mm to (272.3, -25.5), turned to -90 degrees
- moved cch2 204.6 mm to (277.1, -7.42), turned to 180 degrees
- moved eprg1 197.1 mm to (267.8, -3.81), turned to -90 degrees
- moved cen1 194.8 mm to (272.3, -19.9), turned to -90 degrees
- moved ebp1 187.2 mm to (258.3, 10.4), turned to 180 degrees
- moved ebp3 184.0 mm to (253.7, 13.9)
- moved er1 175.0 mm to (232.3, -2.16)
- moved PS1 172.8 mm to (168.0, 25.1)
- moved ebp2 167.1 mm to (236.4, 14.2), turned to 180 degrees
- moved ru2 162.3 mm to (232.3, 8.55), turned to 180 degrees
- moved crp1 160.5 mm to (257.3, 7.15), turned to 90 degrees
- moved ru1 159.1 mm to (232.3, 10.7), turned to 180 degrees
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Connections:
- net /D05_IN1 renamed /D05_IN6
- net /D05_IN2 renamed /D05_IN5
- bridge1 pad 3: /IN220_1N -> /IN220N
- bridge2 pad 3: /IN220_2N -> /IN220N
- cu2 pad 1: unconnected-(cu2-Pad1) -> GND
- in3 pad 4: /D24_IN4 -> /D24_IN3
- in4 pad 4: /D24_IN1 -> /D24_IN4
- in8 pad 4: /D24_IN3 -> /D24_IN1
- mcu1 pad 12: /CHTXD -> /ESP_MCU_RX
- mcu1 pad 13: /CHRXD -> /ESP_MCU_TX
- r12 pad 1: /DI8 -> /DI1
- r16 pad 1: /D24_IN3 -> /D24_IN1
- r30 pad 2: /COM -> /COM1
- r31 pad 2: /COM -> /COM2
- r34 pad 2: /COM -> /COM3
- r35 pad 2: /COM -> /COM4
- r7 pad 1: /D24_IN4 -> /D24_IN3
- r8 pad 1: /D24_IN1 -> /D24_IN4
- relay1 pad 4: unconnected-(relay1-Pad4) -> /NOC
- relay2 pad 1: /RELOUT32 -> /RELOUT22
- relay2 pad 3: /RELOUT31 -> /RELOUT21
- relay2 pad 4: unconnected-(relay2-Pad4) -> /NOC
- relay3 pad 1: /RELOUT42 -> /RELOUT32
- relay3 pad 3: /RELOUT41 -> /RELOUT31
- relay3 pad 4: unconnected-(relay3-Pad4) -> /NOC
- relay4 pad 1: /RELOUT22 -> /RELOUT42
- relay4 pad 3: /RELOUT21 -> /RELOUT41
- relay4 pad 4: unconnected-(relay4-Pad4) -> /NOC
Routing:
- net /ESP_GPIO_0: track 0.00 -> 95.2 mm
- net /DTR: track 0.00 -> 81.3 mm, vias 0 -> 2
- net /ESP_EN: track 0.00 -> 76.8 mm, vias 0 -> 2
- net /RTS: track 0.00 -> 70.5 mm, vias 0 -> 2
- net /+5V: track 0.00 -> 68.9 mm
- net Net-(PS1-+Vout): track 0.00 -> 63.0 mm
- net /ESP_IO2: track 0.00 -> 46.6 mm, vias 0 -> 1
- net /ESP_IO16: track 0.00 -> 42.9 mm, vias 0 -> 1
- net /ESP_IO15: track 0.00 -> 42.0 mm, vias 0 -> 1
- net /ESP_IO7: track 0.00 -> 41.2 mm, vias 0 -> 1
- net /ESP_IO8: track 0.00 -> 40.9 mm, vias 0 -> 1
- net /ESP_IO38: track 0.00 -> 40.6 mm, vias 0 -> 1
- net /ESP_IO6: track 0.00 -> 40.4 mm, vias 0 -> 1
- net /ESP_IO5: track 0.00 -> 38.0 mm, vias 0 -> 1
- net /+3.3V: track 0.00 -> 35.9 mm
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
Commit message: pcb complete; size is the problem
Parts:
- removed r25: 120, Resistor_SMD:R_0805_2012Metric_Pad1.20x1.40mm_HandSolder
- added r6: 120, Resistor_SMD:R_0805_2012Metric_Pad1.20x1.40mm_HandSolder, F.Cu at (202.8, 135.4)
- cm6, cm7, cres1, dr1, dr2, dr3, dr4, qr1, qr2, qr3, qr4, r1, rlb1, rlb2, rlb3, rlb4, rres1: moved to B.Cu
- moved relay1 322.2 mm to (332.4, 8.34)
- moved relay2 322.2 mm to (332.4, 25.3)
- moved relay3 322.1 mm to (332.5, 43.5)
- moved relay4 322.1 mm to (332.5, 60.5)
- moved rb1 317.0 mm to (364.2, 118.3), turned to 180 degrees
- moved rb2 305.2 mm to (363.9, 79.2), turned to 180 degrees
- moved bridge1 285.6 mm to (354.5, 109.8)
- moved aco1 279.7 mm to (315.0, 109.9), turned to 90 degrees
- moved bridge2 278.1 mm to (354.4, 86.8)
- moved cr3 277.8 mm to (330.0, 116.4), turned to 90 degrees
- moved rlb1 277.4 mm to (347.7, 7.74), turned to 180 degrees
- moved cr2 276.9 mm to (329.8, 82.9), turned to -90 degrees
- moved aco2 275.7 mm to (314.7, 89.7), turned to -90 degrees
- moved qr1 273.9 mm to (343.3, 8.65), turned to 180 degrees
- moved rlb2 273.3 mm to (347.8, 24.0), turned to 180 degrees
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Connections:
- net /ADC2 renamed Net-(dz2-K)
- DDO1 pad 1: /DO1 -> /COM1
- DDO1 pad 2: /COM1 -> /DO1
- DDO1 pad 3: /DO2 -> /COM2
- DDO1 pad 4: /COM2 -> /DO2
- DDO1 pad 5: /DO3 -> /COM3
- DDO1 pad 6: /COM3 -> /DO3
- DDO1 pad 7: /DO4 -> /COM4
- DDO1 pad 8: /COM4 -> /DO4
- HS2 pad 6: /D24_IN2 -> /D24_IN1
- U3 pad 7: Net-(U3-B) -> /RS485_B
- in8 pad 4: /D24_IN1 -> /D24_IN2
- iso1 pad 2: /RS485_A -> /RS485_B
- mcu1 pad 14: /AIN1 -> /ADC_IN1
- mcu1 pad 15: /AIN2 -> /ADC_IN2
- mcu1 pad 42: /I2C_SCL -> /MCU_SCL
- mcu1 pad 43: /I2C_SDA -> /MCU_SDA
- r12 pad 1: /DI1 -> /DI2
- r16 pad 1: /D24_IN1 -> /D24_IN2
- r2 pad 1: /DI2 -> /DI1
- r26 pad 1: /RS485_A -> /RS485_B
- r5 pad 1: /D24_IN2 -> /D24_IN1
- relayout1 pad 1: unconnected-(relayout1-Pin_1-Pad1) -> /RELOUT11
- relayout1 pad 2: unconnected-(relayout1-Pin_2-Pad2) -> /RELOUT12
- relayout1 pad 3: unconnected-(relayout1-Pin_3-Pad3) -> /RELOUT21
- relayout1 pad 4: unconnected-(relayout1-Pin_4-Pad4) -> /RELOUT22
- relayout1 pad 5: unconnected-(relayout1-Pin_5-Pad5) -> /RELOUT31
- relayout1 pad 6: unconnected-(relayout1-Pin_6-Pad6) -> /RELOUT32
- relayout1 pad 7: unconnected-(relayout1-Pin_7-Pad7) -> /RELOUT41
- relayout1 pad 8: unconnected-(relayout1-Pin_8-Pad8) -> /RELOUT42
- rsj1 pad 1: /RS485_A -> /RS485_B
Routing:
- net /NOC: track 0.00 -> 75.8 mm
- net MGND: track 0.00 -> 59.4 mm
- net /RELOUT42: track 0.00 -> 47.0 mm
- net Net-(bridge2--): track 0.00 -> 44.6 mm
- net /RELOUT12: track 0.00 -> 43.3 mm
- net Net-(bridge1--): track 0.00 -> 42.7 mm
- net /RELOUT41: track 0.00 -> 41.6 mm
- net /RELOUT32: track 0.00 -> 39.5 mm
- net Net-(cr2-Pad1): track 0.00 -> 32.5 mm
- net Net-(cr3-Pad1): track 0.00 -> 31.8 mm
- net /IN220N: track 0.00 -> 30.5 mm
- net /DI5: track 0.00 -> 29.7 mm
- net /RELOUT22: track 0.00 -> 28.8 mm
- net /RS485_B: track 0.00 -> 26.5 mm
- net /RS485_AO: track 0.00 -> 23.2 mm
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
Commit message: part placement done, semi routed
Parts:
- removed dr3, dr4: 1N4148W, Diode_SMD:D_SOD-123
- removed qr3, qr4: PMBT2222A, Package_TO_SOT_SMD:SOT-23
- removed relay3, relay4: SANYOU_SRD_Form_C, Relay_THT:Relay_SPDT_SANYOU_SRD_Series_Form_C
- removed relayout1: Conn_01x09_Pin, Connector_Molex:Molex_KK-254_AE-6410-09A_1x09_P2.54mm_Vertical
- removed rlb3, rlb4: 1K, Resistor_SMD:R_0805_2012Metric_Pad1.20x1.40mm_HandSolder
- added relo1: Conn_01x05_Pin, Connector_Molex:Molex_KK-254_AE-6410-05A_1x05_P2.54mm_Vertical, F.Cu at (54.5, 96.2)
- CH340, L1, Q1, Q2, U3, U4, U5, aco1, aco2, bridge1, bridge2, c3, c4, c5, c6, c7, cb1, cch1, cch2, cen1, chusb1, cm1, cm2, cm3, cm4, cm5, dz1, dz2, ebj1, ebp2, ebp3, iso1, jadc1, jadc2, out1, out2, out3, out4, qm1, r17, r18, r19, r20, r21, r22, r23, r24, r26, r27, r28, r29, r30, r31, r32, r33, r34, r35, r6, ra1, ra2, ra3, ra4, ra5, ra6, rsj0, rsj1, rsjg1: moved to B.Cu
- moved 220in1 344.2 mm to (6.52, 45.6), turned to 90 degrees
- moved rb1 344.1 mm to (23.4, 70.7), turned to 0 degrees
- moved rb2 335.7 mm to (28.8, 58.1), turned to 0 degrees
- moved bridge1 326.3 mm to (30.8, 68.5), turned to 180 degrees
- moved cr3 321.9 mm to (11.9, 66.5)
- moved r17 317.0 mm to (3.21, 67.4)
- moved aco1 314.5 mm to (4.48, 59.9)
- moved r21 314.0 mm to (4.76, 53.2), turned to 180 degrees
- moved bridge2 313.3 mm to (42.2, 60.3)
- moved r19 311.8 mm to (5.85, 67.3)
- moved rlb2 281.2 mm to (76.1, 96.5), turned to 90 degrees
- moved qr2 276.4 mm to (75.2, 92.0), turned to 90 degrees
- moved dr2 270.8 mm to (75.2, 87.3), turned to -90 degrees
- moved rlb1 270.4 mm to (92.1, 96.3), turned to 90 degrees
- moved cr2 270.1 mm to (60.4, 63.7)
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Routing:
- net /DTR: track 81.3 -> 0.00 mm, vias 2 -> 0
- net /NOC: track 75.8 -> 0.00 mm
- net /RTS: track 70.5 -> 0.00 mm, vias 2 -> 0
- net /+5V: track 73.3 -> 6.03 mm
- net /ESP_EN: track 76.8 -> 13.4 mm, vias 2 -> 0
- net Net-(PS1-+Vout): track 63.0 -> 0.00 mm
- net /RELOUT42: track 47.0 -> 0.00 mm
- net /ESP_IO2: track 46.6 -> 0.00 mm, vias 1 -> 0
- net /RELOUT12: track 43.3 -> 0.00 mm
- net /ESP_IO16: track 42.9 -> 0.00 mm, vias 1 -> 0
- net Net-(bridge2--): track 44.6 -> 2.60 mm
- net /ESP_IO15: track 42.0 -> 0.00 mm, vias 1 -> 0
- net /RELOUT41: track 41.6 -> 0.00 mm
- net /ESP_IO7: track 41.2 -> 0.00 mm, vias 1 -> 0
- net /ESP_IO8: track 40.9 -> 0.00 mm, vias 1 -> 0
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