File: test.kicad_pcb (KiCad board)
At the start: 2 copper layers, 100 x 100 mm, 158 parts, among them Q1 T2N7002AK, Q2 T2N7002AK, SW1 SW_Push, U1 ESP32-S3-WROOM-1, U2 LD1117S33TR_SOT223, U3 SN75176AD, U4 LM321, U5 LM2576HVS-5

Commit message: all done but gnd
Parts:
- removed SW1: SW_Push, Button_Switch_SMD:SW_Push_1P1T_NO_6x6mm_H9.5mm
- added D1: LED, LED_SMD:LED_0805_2012Metric_Pad1.15x1.40mm_HandSolder, F.Cu at (71.5, 29.2)
- added U6: MAX31855KASA, Package_SO:SOIC-8_3.9x4.9mm_P1.27mm, B.Cu at (5.20, 62.8)
- added cx1: 100nF, Capacitor_SMD:C_0805_2012Metric_Pad1.18x1.45mm_HandSolder, B.Cu at (7.63, 68.0)
- added mcur1: Conn_01x02_Pin, Connector_PinHeader_2.54mm:PinHeader_1x02_P2.54mm_Vertical, F.Cu at (56.1, 34.8)
- added mxin1: Screw_Terminal_01x02, TerminalBlock_Phoenix:TerminalBlock_Phoenix_MKDS-1,5-2-5.08_1x02_P5.08mm_Horizontal, F.Cu at (5.27, 53.6)
- added mxj1: 0, Resistor_SMD:R_0805_2012Metric_Pad1.20x1.40mm_HandSolder, B.Cu at (11.5, 64.5)
- added rled1: 1K, Resistor_SMD:R_0805_2012Metric_Pad1.20x1.40mm_HandSolder, F.Cu at (70.2, 36.6)
- cm1, rf2: moved to F.Cu
- moved cm5 18.3 mm to (68.1, 37.6)
- moved cm4 18.0 mm to (70.2, 37.6)
- moved cm3 17.8 mm to (72.3, 37.6)
- moved r5 14.3 mm to (38.8, 43.2), turned to 180 degrees
- moved cm2 13.6 mm to (69.5, 41.5)
- moved pwrs1 12.9 mm to (13.5, 54.1), turned to 90 degrees
- moved Ds1 11.6 mm to (19.5, 83.0)
- moved rf2 10.3 mm to (91.5, 57.5), turned to -90 degrees
- moved C2 10.0 mm to (18.0, 70.4)
- moved cr2 8.20 mm to (38.0, 55.4)
- moved crs2 6.39 mm to (14.7, 62.4)
- moved cm7 6.33 mm to (45.3, 43.4)
- moved cr3 6.11 mm to (26.6, 59.0)
- moved crs1 5.91 mm to (24.7, 67.8)
- moved BAT1 5.77 mm to (36.3, 15.0)
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Connections:
- espio1 pad 21: /3.3V -> /+3.3V
- mcu1 pad 32: unconnected-(mcu1-PA11-Pad32) -> /MXCS
- mcu1 pad 4: unconnected-(mcu1-PC15-Pad4) -> /LED
- relo1 pad 1: /RELOUT12 -> /RELOUT22
- relo1 pad 2: /RELOUT11 -> /RELOUT21
- relo1 pad 3: /RELOUT22 -> /RELOUT12
- relo1 pad 4: /RELOUT21 -> /RELOUT11
Routing:
- net /+3.3V: track 4.93 -> 709.6 mm, vias 0 -> 13
- net /+5V: track 0.00 -> 519.1 mm, vias 0 -> 4
- net /MXCS: track 0.00 -> 159.1 mm, vias 0 -> 1
- net IGND: track 0.00 -> 153.6 mm, vias 0 -> 5
- net /SO: track 14.8 -> 149.8 mm, vias 0 -> 1
- net /SCK: track 24.9 -> 125.8 mm, vias 0 -> 1
- net AGND: track 0.00 -> 64.1 mm, vias 0 -> 10
- net /VBAT: track 50.0 -> 77.6 mm
- net /LED: track 0.00 -> 24.8 mm
- net /RELOUT22: track 30.2 -> 52.1 mm
- net Net-(Ds1-K): track 38.2 -> 58.0 mm
- net /D24_IN1: track 97.3 -> 79.0 mm
- net Net-(U6-T-): track 0.00 -> 17.2 mm
- net /+24V: track 213.1 -> 198.5 mm
- net Net-(dr2-A): track 13.5 -> 25.7 mm
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- added copper zone on B.Cu, net AGND
- added copper zone on F.Cu, net AGND

Commit message: final version. needs cleanup and marckage
Parts:
- moved din1 1.00 mm to (5.25, 29.3)
- moved cm1 0.52 mm to (78.0, 50.5)
- moved qm1 0.40 mm to (21.8, 31.0)
- moved ce2 0.15 mm to (58.0, 2.05)
- moved ce1 0.11 mm to (61.1, 1.99)
- turned ra3 to 0 degrees
Routing:
- net /+5V: track 519.1 -> 626.8 mm
- net MGND: track 90.8 -> 85.1 mm
- net /RS485_AO: track 81.7 -> 77.2 mm
- net /SO: track 149.8 -> 145.5 mm
- net /MCU_RX: track 181.0 -> 177.2 mm
- net /MDO2: track 151.2 -> 147.8 mm
- net AGND: track 64.1 -> 61.1 mm, vias 10 -> 6
- net /rlo1: track 60.4 -> 57.9 mm
- net Net-(bridge1--): track 73.3 -> 71.0 mm
- net /MDO3: track 151.4 -> 149.3 mm
- net /MDO1: track 148.6 -> 146.7 mm
- net /MDO4: track 140.2 -> 138.4 mm
- net /RS485_A: track 16.1 -> 14.5 mm
- net /rlo2: track 50.6 -> 49.1 mm
- net Net-(U4-+): track 5.23 -> 6.67 mm
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- added copper zone on B.Cu, net GND
- added copper zone on F.Cu, net GND

Commit message: polygon and solder mask complete. DRC complete
Routing:
- net /rlo1: track 57.9 -> 61.5 mm
- net /+3.3V: track 709.5 -> 712.9 mm
- net IGND: track 154.9 -> 152.2 mm
- net /ESP_IO4: track 31.3 -> 29.3 mm
- net /ESP_IO5: track 33.1 -> 31.5 mm
- net /ESP_IO7: track 34.4 -> 32.9 mm
- net AGND: track 61.1 -> 59.6 mm, vias 6 -> 7
- net /ESP_IO6: track 32.9 -> 31.5 mm
- net Net-(dr2-A): track 24.9 -> 23.8 mm
- net /rlo2: track 49.1 -> 50.1 mm
- net Net-(cr2-Pad1): track 44.5 -> 43.6 mm
- net Net-(usb1-Pin_1): track 11.2 -> 12.0 mm
- net /ESP_IO15: track 34.7 -> 33.9 mm
- net Net-(bridge1--): track 71.0 -> 70.4 mm
- net Net-(D1-A): track 6.90 -> 6.25 mm
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
Commit message: first version to print
Parts:
- added G***: LOGO, LOGO, F.Cu at (35.0, 31.1)
- Relay Out: renamed from relo1
- renumbered pwr1 to 24in, din1 to DIN, ebt1 to IO3S, chusb1 to espprg, modout1 to modbus, pwrs1 to pwrsel, prg1 to stprg, mxin1 to thermo
Routing:
- net (no net): vias 0 -> 3
Other:
- board text added: "+24V"
- board text added: "1"
- board text added: "2"
- board text added: "220V IN (L2 - N - L1)"
- board text added: "220V POWER"
- board text added: "3"
- board text added: "3V3"
- board text added: "4"
- board text added: "5"
- board text added: "6"
- board text added: "A"
- board text added: "AC24"
- board text added: "AIN"
- board text added: "B"
- board text added: "C1"
- board text added: "C11"
- board text added: "C12"
- board text added: "C2"
- board text added: "C21"
- board text added: "C22"
- board text added: "C3"
- board text added: "C4"
- board text added: "CLK"
- board text added: "Cx1"
- board text added: "Cx2"
- board text added: "D+"
- board text added: "D-"
- board text added: "D1"
- board text added: "D2"
- board text added: "D3"
- board text added: "D4"
- board text added: "DIO"
- board text added: "EXT24"
- board text added: "G"
- board text added: "GND"
- board text added: "L ~ N"
- board text added: "N1"
- board text added: "N2"
- board text added: "Nx"
- board text added: "PD01-BLE"
- board text added: "RES"
- board text added: "RESET"
- board text added: "SCL"
- board text added: "SDA"
- board text added: "T+"
- board text added: "T-"
