File: test.kicad_sch (KiCad schematic)
At the start: 81 parts, among them Q1 T2N7002AK, Q2 T2N7002AK, SW1 SW_Push, U1 ESP32-S3-WROOM-1, U2 LD1117S33TR_SOT223, U3 AT45DB161D-SU

Commit message: schematic almost complete
Parts:
- removed opt1, opt10, opt11, opt12, opt13, opt14, opt15, opt16, opt2, opt3, opt4, opt5, opt6, opt7, opt8, opt9: PC817, Package_DIP:DIP-4_W7.62mm_SMDSocket_SmallPads, symbol Isolator:PC817
- removed rel2, rel3, rel4: SANYOU_SRD_Form_C, Relay_THT:Relay_SPDT_SANYOU_SRD_Series_Form_C, symbol Relay:SANYOU_SRD_Form_C
- added U3: SN75176AD, Package_SO:SOIC-8_3.9x4.9mm_P1.27mm, symbol Interface_UART:SN75176AD
- added U4, U5: LM321, Package_TO_SOT_SMD:SOT-23-5, symbol Amplifier_Operational:LM321
- added aco1, aco2, in1, in2, in3, in4, in5, in6, in7, in8, out1, out2, out3, out4: PC817, Package_DIP:DIP-4_W7.62mm_SMDSocket_SmallPads, symbol Isolator:PC817
- added bridge1, bridge2: MB1S, Diode_SMD:Diode_Bridge_OnSemi_SDIP-4L, symbol Diode_Bridge:DF01S1
- added c3, cf1: 100nF, Capacitor_SMD:C_0805_2012Metric_Pad1.18x1.45mm_HandSolder, symbol Device:C
- added cr2, cr3: C_Polarized, Capacitor_THT:CP_Axial_L30.0mm_D10.0mm_P35.00mm_Horizontal, symbol Device:C_Polarized
- added di1, di2, di3, di4, di5, di6, di7, di8, dr1, dr2, dr3, dr4: 1N4148W, Diode_SMD:D_SOD-123, symbol Diode:1N4148W
- added dz1, dz2: D_Zener, Diode_SMD:D_MiniMELF_Handsoldering, symbol Device:D_Zener
- added qm1, qr1, qr2, qr3, qr4: PMBT2222A, Package_TO_SOT_SMD:SOT-23, symbol Transistor_BJT:PMBT2222A
- added r1, r11, r12, r2, r3, r4: 7.5K, Resistor_SMD:R_1206_3216Metric_Pad1.30x1.75mm_HandSolder, symbol Device:R_US
- added r10: 2.8K, Resistor_SMD:R_1206_3216Metric_Pad1.30x1.75mm_HandSolder, symbol Device:R_US
- added r13, r14, r15, r16, r5, r6, r7, r8: 680, Resistor_SMD:R_0805_2012Metric_Pad1.20x1.40mm_HandSolder, symbol Device:R_US
- added r17, r18, rlb1, rlb2, rlb3, rlb4: 1K, Resistor_SMD:R_0805_2012Metric_Pad1.20x1.40mm_HandSolder, symbol Device:R_US
- added r19, r20: 560, Resistor_SMD:R_0805_2012Metric_Pad1.20x1.40mm_HandSolder, symbol Device:R_US
- added r21, r22, ra1, ra2, rf1, rf2: 100K, Resistor_SMD:R_0805_2012Metric_Pad1.20x1.40mm_HandSolder, symbol Device:R_US
- added r23, r24, r26, r27: 10K, Resistor_SMD:R_0805_2012Metric_Pad1.20x1.40mm_HandSolder, symbol Device:R_US
- added r25: 120, Resistor_SMD:R_0805_2012Metric_Pad1.20x1.40mm_HandSolder, symbol Device:R_US
- added r28, r29, r32, r33: 2.7K, Resistor_SMD:R_1206_3216Metric_Pad1.30x1.75mm_HandSolder, symbol Device:R_US
- added r30, r31, r34, r35: 3.3K, Resistor_SMD:R_0805_2012Metric_Pad1.20x1.40mm_HandSolder, symbol Device:R_US
- added r9: 2.5K, Resistor_SMD:R_1206_3216Metric_Pad1.30x1.75mm_HandSolder, symbol Device:R_US
- added ra3, ra4: 33K, Resistor_SMD:R_0805_2012Metric_Pad1.20x1.40mm_HandSolder, symbol Device:R_US
- added ra5, ra6: 68, Resistor_SMD:R_0805_2012Metric_Pad1.20x1.40mm_HandSolder, symbol Device:R_US
- added rb1, rb2: 100K, Resistor_THT:R_Axial_DIN0414_L11.9mm_D4.5mm_P20.32mm_Horizontal, symbol Device:R
- added relay2, relay3, relay4: SANYOU_SRD_Form_C, Relay_THT:Relay_SPDT_SANYOU_SRD_Series_Form_C, symbol Relay:SANYOU_SRD_Form_C
- renumbered U3 to flash1, rel1 to relay1
Connections:
- net +3.3V: now also flash1.6 (VCC), cf1.2, r13.2, r14.2, r15.2, r16.2, r21.2, r22.2, r5.2, r6.2, r7.2, r8.2, rf1.1, rf2.1
- net +5V: now also relay1.5, U3.8 (VCC), U4.5 (V+), U5.5 (V+), c3.2, dr1.1 (K), dr2.1 (K), dr3.1 (K), dr4.1 (K), r23.2, r26.2, relay2.5, relay3.5, relay4.5
- net AGND: now also U4.2 (V-), U5.2 (V-), dz1.2 (A), dz2.2 (A), ra3.1, ra4.1
- net GND: now also flash1.7 (GND), U3.5 (GND), aco1.3, aco2.3, c3.1, cf1.1, in1.3, in2.3, in3.3, in4.3, in5.3, in6.3, in7.3, in8.3, out1.2, out2.2, out3.2, out4.2, qr1.2 (E), qr2.2 (E), qr3.2 (E), qr4.2 (E), r24.2, r27.1
- net SI: now reaches flash1.1 (SI)
- net SCK: now reaches flash1.2 (SCK)
- net FRES: now reaches flash1.3 (~{RESET})
- net FRES: now also rf2.2
- net CS: now reaches flash1.4 (~{CS})
- net at flash1.5 (~{WP}): now also rf1.2
- net SO: now reaches flash1.8 (SO)
- net at relay1.2: now also dr1.2 (A), qr1.3 (C)
- new net: U5.3 (-), U5.4, ra6.1
- new net: dr4.2 (A), qr4.3 (C), relay4.2
- new net: di4.1 (K), in4.1, r4.2
- new net: in4.4, r8.1
- new net: out4.1, r33.2
- new net: out4.4, r35.1
- new net: qr1.1 (B), rlb1.2
- new net: U4.1 (+), ra1.2, ra3.2
- new net: U4.3 (-), U4.4, ra5.1
- new net: aco2.1, r20.1
- new net: r18.2, r20.2, rb2.2
- new net: bridge2.1 (+), cr3.1, rb2.1
- new net: aco2.2, bridge2.2 (-), cr3.2, r18.1
- new net: di2.1 (K), in2.1, r2.2
- new net: in2.4, r6.1
- new net: dr2.2 (A), qr2.3 (C), relay2.2
- new net: aco1.1, r19.1
- new net: aco1.2, bridge1.2 (-), cr2.2, r17.1
- new net: aco1.4, r21.1
- new net: di3.1 (K), in3.1, r3.2
- new net: in3.4, r7.1
- new net: di5.1 (K), in5.1, r9.2
- new net: in7.4, r15.1
- new net: out1.1, r28.2
- new net: di8.1 (K), in8.1, r12.2
- new net: bridge1.1 (+), cr2.1, rb1.1
- new net: in5.4, r13.1
- new net: di1.1 (K), in1.1, r1.2
- new net: out1.4, r30.1
- new net: qr2.1 (B), rlb2.2
- new net: out2.4, r31.1
- new net: di7.1 (K), in7.1, r11.2
- new net: in1.4, r5.1
- new net: dr3.2 (A), qr3.3 (C), relay3.2
- new net: r17.2, r19.2, rb1.2
- new net: qr3.1 (B), rlb3.2
- new net: U5.1 (+), ra2.2, ra4.2
- new net: out3.4, r34.1
- new net: in6.4, r14.1
- new net: di6.1 (K), in6.1, r10.2
- new net: qm1.2 (E), r24.1
- new net: in8.4, r16.1
- new net: qr4.1 (B), rlb4.2
- new net: out3.1, r32.2
- new net: U3.2 (~{RE}), U3.3 (DE), qm1.3 (C), r23.1
- new net: U3.7 (B), r25.2
- new net: out2.1, r29.2
- new net: aco2.4, r22.1
- new net ADC1: dz1.1 (K), ra5.2
- new net ADC2: dz2.1 (K), ra6.2
- new net AIN1: ra1.1
- new net AIN2: ra2.1
- new net COM: r30.2, r31.2, r34.2, r35.2
- new net DI1: r1.1
- new net DI2: r2.1
- new net DI3: r3.1
- new net DI4: r4.1
- new net DI5: r9.1
- new net DI6: r10.1
- new net DI7: r11.1
- new net DI8: r12.1
- new net DO1: out1.3
- new net DO2: out3.3
- new net DO3: out2.3
- new net DO4: out4.3
- new net IGND: di1.2 (A), di2.2 (A), di3.2 (A), di4.2 (A), di5.2 (A), di6.2 (A), di7.2 (A), di8.2 (A), in1.2, in2.2, in3.2, in4.2, in5.2, in6.2, in7.2, in8.2
- new net IN220_1L: bridge1.4
- new net IN220_1N: bridge1.3
- new net IN220_2L: bridge2.4
- new net IN220_2N: bridge2.3
- new net MCU_RX: U3.1 (R)
- new net MCU_TX: U3.4 (D)
- new net MDO1: r28.1, r29.1, r32.1, r33.1
- new net RS485_A: U3.6 (A), r25.1, r26.1, r27.2
- new net RS_SEL: qm1.1 (B)
- new net rlo1: rlb1.1
- new net rlo2: rlb2.1
- new net rlo3: rlb3.1
- new net rlo4: rlb4.1
- no-connect marks 13 -> 12
Other:
- note added: "12-24V"
- note added: "220V INPUTS"
- note added: "5V"
- note added: "ANALOG INPUTS"
- note added: "DIGITAL INPUTS"
- note added: "Digital Output"
- note added: "MODBUS"
- note added: "Relay Output"
- moved on the sheet: BAT1, L0, SW1, cb1, chse1, chse2, clse1, clse2, cm1, cm2, cm3, cm4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

Commit message: schematic complete
Parts:
- removed #u31: STM32F031C6Tx, Package_QFP:LQFP-48_7x7mm_P0.5mm, symbol MCU_ST_STM32F0:STM32F031C6Tx
- removed L0: L_Ferrite, Inductor_SMD:L_0805_2012Metric_Pad1.05x1.20mm_HandSolder, symbol Device:L_Ferrite
- removed di1, di7: 1N4148W, Diode_SMD:D_SOD-123, symbol Diode:1N4148W
- removed in1, in2, in5, in7: PC817, Package_DIP:DIP-4_W7.62mm_SMDSocket_SmallPads, symbol Isolator:PC817
- removed r11: 7.5K, Resistor_SMD:R_1206_3216Metric_Pad1.30x1.75mm_HandSolder, symbol Device:R_US
- removed r13, r15, r6: 680, Resistor_SMD:R_0805_2012Metric_Pad1.20x1.40mm_HandSolder, symbol Device:R_US
- added HS1, HS2: 6N137, Package_DIP:DIP-8_W7.62mm, symbol Isolator:6N137
- added L1: L_Ferrite, Inductor_SMD:L_0805_2012Metric_Pad1.05x1.20mm_HandSolder, symbol Device:L_Ferrite
- added OLED1, Sensor1: Conn_01x04_Pin, Connector_Molex:Molex_KK-254_AE-6410-04A_1x04_P2.54mm_Vertical, symbol Connector:Conn_01x04_Pin
- added c4, c5, cm6, cm7: 100nF, Capacitor_SMD:C_0805_2012Metric_Pad1.18x1.45mm_HandSolder, symbol Device:C
- added i2c1, i2c2: 100K, Resistor_SMD:R_0805_2012Metric_Pad1.20x1.40mm_HandSolder, symbol Device:R_US
- added jadc1, jadc2: 0, Resistor_SMD:R_0805_2012Metric_Pad1.20x1.40mm_HandSolder, symbol Device:R
- cr2, cr3: footprint Capacitor_THT:CP_Axial_L30.0mm_D10.0mm_P35.00mm_Horizontal -> Capacitor_THT:CP_Radial_D22.0mm_P10.00mm_SnapIn
- r1: value 7.5K -> 680; footprint Resistor_SMD:R_1206_3216Metric_Pad1.30x1.75mm_HandSolder -> Resistor_SMD:R_0805_2012Metric_Pad1.20x1.40mm_HandSolder
- r2: value 7.5K -> 2.2K
- r9: value 2.5K -> 560
- ra1, ra2: value 100K -> 68K
Connections:
- net +3.3V: now also prg1.5 (Pin_5), OLED1.3 (Pin_3), Sensor1.4 (Pin_4), i2c1.1, i2c2.1; no longer r5.2
- net +5V: now also r1.2, r5.2, HS1.8 (VCC), HS2.8 (VCC), c4.1, c5.1, cm6.1, cm7.1
- net ADC2: now also jadc2.1
- net AGND: now also L1.2, c4.2, c5.2
- net AIN1: now also mcu1.14 (PA4)
- net AIN2: now also mcu1.15 (PA5)
- net CHRXD: now also mcu1.13 (PA3)
- net CHTXD: now also mcu1.12 (PA2)
- net CS: now also mcu1.25 (PB12)
- net DO2: now also out2.3; no longer out3.3
- net DO3: now also out3.3; no longer out2.3
- net GND: now also U2.1 (GND), HS1.5 (GND), HS2.5 (GND), L1.1, OLED1.4 (Pin_4), Sensor1.1 (Pin_1), cm6.2, cm7.2
- net IGND: now also HS1.3 (C), HS2.3 (C)
- net MDO1: no longer r29.1, r32.1, r33.1
- net SCK: now also mcu1.26 (PB13)
- net SI: now also mcu1.28 (PB15)
- net SO: now also mcu1.27 (PB14)
- net RELOUT22: now reaches relay4.1
- net RELOUT21: now reaches relay4.3
- net D24_IN1: now reaches in4.4, r8.1
- net at r18.2, r20.2, rb2.2: now also cr2.1
- net at bridge2.1 (+), rb2.1: no longer cr3.1
- net at aco2.2, bridge2.2 (-), r18.1: now also cr2.2; no longer cr3.2
- net at di2.1 (K), r2.2: now also HS2.2 (A)
- net RELOUT12: now reaches relay1.1
- net RELOUT11: now reaches relay1.3
- net at aco1.2, bridge1.2 (-), r17.1: now also cr3.2; no longer cr2.2
- net D220_IN1: now reaches aco1.4, r21.1
- net D24_IN4: now reaches in3.4, r7.1
- net at di5.1 (K), r9.2: now also HS1.2 (A)
- net UART1_TX: now reaches mcu1.30 (PA9)
- net UART1_RX: now reaches mcu1.31 (PA10)
- net I2C_SCL: now reaches mcu1.42 (PB6)
- net I2C_SDA: now reaches mcu1.43 (PB7)
- net at bridge1.1 (+), rb1.1: no longer cr2.1
- net D24_IN2: now reaches r5.1
- net D24_IN2: now also HS2.6 (VO)
- net at r17.2, r19.2, rb1.2: now also cr3.1
- net D05_IN1: now reaches in6.4, r14.1
- net D24_IN3: now reaches in8.4, r16.1
- net RELOUT32: now reaches relay2.1
- net RELOUT31: now reaches relay2.3
- net RELOUT42: now reaches relay3.1
- net RELOUT41: now reaches relay3.3
- net D220_IN2: now reaches aco2.4, r22.1
- net ADC1: no longer names the net of dz1.1 (K), ra5.2
- net ADC1: now also jadc1.1
- net DI1 renamed D05_IN2
- net D05_IN2: now also HS1.6 (VO)
- net FRES: no longer names the net of flash1.3 (~{RESET}), rf2.2
- net SWO: no longer names the net of mcu1.39 (PB3)
- net SWO: no longer prg1.5 (Pin_5)
- new net ADC_IN1: jadc1.2
- new net ADC_IN2: jadc2.2
- new net MCU_SCL: OLED1.2 (Pin_2), Sensor1.3 (Pin_3), i2c2.2
- new net MCU_SDA: OLED1.1 (Pin_1), Sensor1.2 (Pin_2), i2c1.2
- new net MDO2: r29.1
- new net MDO3: r32.1
- new net MDO4: r33.1
- no-connect marks 12 -> 18
Other:
- moved on the sheet: U3, c3, di3, di4, in3, in4, qm1, r17, r18, r23, r24, r25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

Commit message: finished power and esp32 in pcb
Parts:
- removed C1: 100nF, Capacitor_SMD:C_0805_2012Metric_Pad1.18x1.45mm_HandSolder, symbol Device:C
- removed C2: 10uF, Capacitor_SMD:C_0805_2012Metric_Pad1.18x1.45mm_HandSolder, symbol Device:C
- removed ESP_GPIO1: Conn_02x11_Odd_Even, Connector_PinHeader_2.00mm:PinHeader_2x11_P2.00mm_Vertical, symbol Connector_Generic:Conn_02x11_Odd_Even
- added 220in1, MODBUS1: Screw_Terminal_01x03, TerminalBlock:TerminalBlock_Altech_AK300-3_P5.00mm, symbol Connector:Screw_Terminal_01x03
- added AIN1: Conn_01x03_Pin, Connector_Molex:Molex_KK-254_AE-6410-03A_1x03_P2.54mm_Vertical, symbol Connector:Conn_01x03_Pin
- added C1, C2: C_Polarized, Capacitor_THT:CP_Radial_D4.0mm_P1.50mm, symbol Device:C_Polarized
- added DDO1: Conn_01x08_Socket, Connector_Molex:Molex_KK-254_AE-6410-08A_1x08_P2.54mm_Vertical, symbol Connector:Conn_01x08_Socket
- added acin1: Screw_Terminal_01x02, TerminalBlock_MetzConnect:TerminalBlock_MetzConnect_Type011_RT05502HBWC_1x02_P5.00mm_Horizontal, symbol Connector:Screw_Terminal_01x02
- added c6, c7: 100nF, Capacitor_SMD:C_0805_2012Metric_Pad1.18x1.45mm_HandSolder, symbol Device:C
- added din1: Conn_01x07_Pin, Connector_Molex:Molex_KK-254_AE-6410-07A_1x07_P2.54mm_Vertical, symbol Connector:Conn_01x07_Pin
- added espio1: Conn_02x11_Odd_Even, Connector_PinHeader_2.00mm:PinHeader_2x11_P2.00mm_Vertical, symbol Connector_Generic:Conn_02x11_Odd_Even
- added iso1: ADuM1201BR, Package_SO:SOIC-8_3.9x4.9mm_P1.27mm, symbol Isolator:ADuM1201BR
- added iso5: Conn_01x04_Pin, Connector_Molex:Molex_KK-254_AE-6410-04A_1x04_P2.54mm_Vertical, symbol Connector:Conn_01x04_Pin
- added relayout1: Conn_01x09_Pin, Connector_Molex:Molex_KK-254_AE-6410-09A_1x09_P2.54mm_Vertical, symbol Connector:Conn_01x09_Pin
- added rsj0, rsj1, rsjg1: 0, Resistor_SMD:R_0805_2012Metric_Pad1.20x1.40mm_HandSolder, symbol Device:R
Connections:
- net IN220_2N is gone; now on net IN220N: bridge2.3
- net +3.3V: now also C2.1
- net +5V: now also C1.1, c6.2, iso1.1 (VDD1), iso5.2 (Pin_2)
- net 3.3V: now also espio1.21 (Pin_21)
- net AGND: now also AIN1.2 (Pin_2)
- net AIN1: now also AIN1.1 (Pin_1)
- net AIN2: now also AIN1.3 (Pin_3)
- net CHRXD: no longer mcu1.13 (PA3)
- net CHTXD: no longer mcu1.12 (PA2)
- net D24_IN1: now also in8.4, r16.1; no longer in4.4, r8.1
- net D24_IN3: now also in3.4, r7.1; no longer in8.4, r16.1
- net D24_IN4: now also in4.4, r8.1; no longer in3.4, r7.1
- net DI2: now also din1.2 (Pin_2)
- net DI3: now also din1.3 (Pin_3)
- net DI4: now also din1.4 (Pin_4)
- net DI5: now also din1.5 (Pin_5)
- net DI6: now also din1.6 (Pin_6)
- net DO1: now also DDO1.1 (Pin_1)
- net DO2: now also DDO1.3 (Pin_3)
- net DO3: now also DDO1.5 (Pin_5)
- net DO4: now also DDO1.7 (Pin_7)
- net ESP_IO1: now also espio1.20 (Pin_20)
- net ESP_IO10: now also espio1.4 (Pin_4)
- net ESP_IO11: now also espio1.6 (Pin_6)
- net ESP_IO12: now also espio1.8 (Pin_8)
- net ESP_IO13: now also espio1.10 (Pin_10)
- net ESP_IO14: now also espio1.12 (Pin_12)
- net ESP_IO15: now also espio1.9 (Pin_9)
- net ESP_IO16: now also espio1.11 (Pin_11)
- net ESP_IO2: now also espio1.17 (Pin_17)
- net ESP_IO21: now also espio1.14 (Pin_14)
- net ESP_IO38: now also espio1.15 (Pin_15)
- net ESP_IO4: now also espio1.1 (Pin_1)
- net ESP_IO47: now also espio1.16 (Pin_16)
- net ESP_IO48: now also espio1.18 (Pin_18)
- net ESP_IO5: now also espio1.3 (Pin_3)
- net ESP_IO6: now also espio1.5 (Pin_5)
- net ESP_IO7: now also espio1.7 (Pin_7)
- net ESP_IO8: now also espio1.13 (Pin_13)
- net ESP_IO9: now also espio1.2 (Pin_2)
- net ESP_MCU_RX: now also mcu1.12 (PA2)
- net ESP_MCU_TX: now also mcu1.13 (PA3)
- net GND: now also cu2.1, C1.2, C2.2, c6.1, espio1.22 (Pin_22), iso1.4 (GND1), iso5.1 (Pin_1), rsjg1.1
- net IGND: now also din1.7 (Pin_7)
- net IN220_1L: now also 220in1.3 (Pin_3)
- net IN220_2L: now also 220in1.1 (Pin_1)
- net L: now also acin1.2 (Pin_2)
- net N: now also acin1.1 (Pin_1)
- net RELOUT21: now also relay2.3; no longer relay4.3
- net RELOUT22: now also relay2.1; no longer relay4.1
- net RELOUT31: now also relay3.3; no longer relay2.3
- net RELOUT32: now also relay3.1; no longer relay2.1
- net RELOUT41: now also relay4.3; no longer relay3.3
- net RELOUT42: now also relay4.1; no longer relay3.1
- net RS485_A: now also iso1.2 (VOA), iso1.3 (VIB), rsj0.1, rsj1.1
- net NOC: now reaches relay4.4
- net NOC: now also relay1.4, relay2.4, relay3.4, relayout1.9 (Pin_9)
- removed net COM: r30.2, r31.2, r34.2, r35.2
- net D05_IN1 renamed D05_IN6
- net D05_IN2 renamed D05_IN5
- net DI8 renamed DI1
- net DI1: now also din1.1 (Pin_1)
- net IN220_1N renamed IN220N
- net IN220N: now also 220in1.2 (Pin_2)
- new net +M5V: c7.2, iso1.8 (VDD2), iso5.4 (Pin_4)
- new net COM1: DDO1.2 (Pin_2), r30.2
- new net COM2: DDO1.4 (Pin_4), r31.2
- new net COM3: DDO1.6 (Pin_6), r34.2
- new net COM4: DDO1.8 (Pin_8), r35.2
- new net MGND: MODBUS1.3 (Pin_3), c7.1, iso1.5 (GND2), iso5.3 (Pin_3), rsjg1.2
- new net RS485_AO: MODBUS1.1 (Pin_1), iso1.6 (VOB), rsj0.2
- new net RS485_BO: MODBUS1.2 (Pin_2), iso1.7 (VIA), rsj1.2
Other:
- note added: "5v TO 5V CONVERTOR"
- moved on the sheet: U3, c3, qm1, r23, r24, r25, r26, r27

Commit message: pcb complete; size is the problem
Parts:
- removed r25: 120, Resistor_SMD:R_0805_2012Metric_Pad1.20x1.40mm_HandSolder, symbol Device:R_US
- added r6: 120, Resistor_SMD:R_0805_2012Metric_Pad1.20x1.40mm_HandSolder, symbol Device:R_US
Connections:
- net I2C_SCL is gone; now on net MCU_SCL: mcu1.42 (PB6)
- net I2C_SDA is gone; now on net MCU_SDA: mcu1.43 (PB7)
- net ADC_IN1: now also mcu1.14 (PA4)
- net ADC_IN2: now also mcu1.15 (PA5)
- net AIN1: no longer mcu1.14 (PA4)
- net AIN2: no longer mcu1.15 (PA5)
- net COM1: now also DDO1.1 (Pin_1); no longer DDO1.2 (Pin_2)
- net COM2: now also DDO1.3 (Pin_3); no longer DDO1.4 (Pin_4)
- net COM3: now also DDO1.5 (Pin_5); no longer DDO1.6 (Pin_6)
- net COM4: now also DDO1.7 (Pin_7); no longer DDO1.8 (Pin_8)
- net D24_IN1: now also HS2.6 (VO), r5.1; no longer in8.4, r16.1
- net D24_IN2: now also in8.4, r16.1; no longer HS2.6 (VO), r5.1
- net DI1: now also r2.1; no longer r12.1
- net DI2: now also r12.1; no longer r2.1
- net DO1: now also DDO1.2 (Pin_2); no longer DDO1.1 (Pin_1)
- net DO2: now also DDO1.4 (Pin_4); no longer DDO1.3 (Pin_3)
- net DO3: now also DDO1.6 (Pin_6); no longer DDO1.5 (Pin_5)
- net DO4: now also DDO1.8 (Pin_8); no longer DDO1.7 (Pin_7)
- net RELOUT11: now also relayout1.1 (Pin_1)
- net RELOUT12: now also relayout1.2 (Pin_2)
- net RELOUT21: now also relayout1.3 (Pin_3)
- net RELOUT22: now also relayout1.4 (Pin_4)
- net RELOUT31: now also relayout1.5 (Pin_5)
- net RELOUT32: now also relayout1.6 (Pin_6)
- net RELOUT41: now also relayout1.7 (Pin_7)
- net RELOUT42: now also relayout1.8 (Pin_8)
- net RS485_A: now also r6.2; no longer iso1.2 (VOA), r26.1, rsj1.1
- net RS485_B: now reaches U3.7 (B)
- net RS485_B: now also iso1.2 (VOA), r26.1, rsj1.1, r6.1
- net ADC2: no longer names the net of dz2.1 (K), jadc2.1, ra6.2
Other:
- moved on the sheet: r26, relayout1

Commit message: part placement done, semi routed
Parts:
- removed dr3, dr4: 1N4148W, Diode_SMD:D_SOD-123, symbol Diode:1N4148W
- removed qr3, qr4: PMBT2222A, Package_TO_SOT_SMD:SOT-23, symbol Transistor_BJT:PMBT2222A
- removed relay3, relay4: SANYOU_SRD_Form_C, Relay_THT:Relay_SPDT_SANYOU_SRD_Series_Form_C, symbol Relay:SANYOU_SRD_Form_C
- removed relayout1: Conn_01x09_Pin, Connector_Molex:Molex_KK-254_AE-6410-09A_1x09_P2.54mm_Vertical, symbol Connector:Conn_01x09_Pin
- removed rlb3, rlb4: 1K, Resistor_SMD:R_0805_2012Metric_Pad1.20x1.40mm_HandSolder, symbol Device:R_US
- added relo1: Conn_01x05_Pin, Connector_Molex:Molex_KK-254_AE-6410-05A_1x05_P2.54mm_Vertical, symbol Connector:Conn_01x05_Pin
Connections:
- net NOC: now also relo1.5 (Pin_5)
- net RELOUT11: now also relo1.1 (Pin_1)
- net RELOUT12: now also relo1.2 (Pin_2)
- net RELOUT21: now also relo1.3 (Pin_3)
- net RELOUT22: now also relo1.4 (Pin_4)

Commit message: except DI1-4 all other logics are ok
Parts:
- removed MODBUS1: Screw_Terminal_01x03, TerminalBlock:TerminalBlock_Altech_AK300-3_P5.00mm, symbol Connector:Screw_Terminal_01x03
- removed Sensor1: Conn_01x04_Pin, Connector_Molex:Molex_KK-254_AE-6410-04A_1x04_P2.54mm_Vertical, symbol Connector:Conn_01x04_Pin
- removed U5: LM321, Package_TO_SOT_SMD:SOT-23-5, symbol Amplifier_Operational:LM321
- removed c5: 100nF, Capacitor_SMD:C_0805_2012Metric_Pad1.18x1.45mm_HandSolder, symbol Device:C
- removed dz2: D_Zener, Diode_SMD:D_MiniMELF_Handsoldering, symbol Device:D_Zener
- removed jadc2: 0, Resistor_SMD:R_0805_2012Metric_Pad1.20x1.40mm_HandSolder, symbol Device:R
- removed ra2: 68K, Resistor_SMD:R_0805_2012Metric_Pad1.20x1.40mm_HandSolder, symbol Device:R_US
- removed ra4: 33K, Resistor_SMD:R_0805_2012Metric_Pad1.20x1.40mm_HandSolder, symbol Device:R_US
- removed ra6: 68, Resistor_SMD:R_0805_2012Metric_Pad1.20x1.40mm_HandSolder, symbol Device:R_US
- removed relo1: Conn_01x05_Pin, Connector_Molex:Molex_KK-254_AE-6410-05A_1x05_P2.54mm_Vertical, symbol Connector:Conn_01x05_Pin
- added modout1: Screw_Terminal_01x03, TerminalBlock_Phoenix:TerminalBlock_Phoenix_MKDS-1,5-3-5.08_1x03_P5.08mm_Horizontal, symbol Connector:Screw_Terminal_01x03
- added relo1: Conn_01x06_Pin, Connector_Molex:Molex_KK-254_AE-6410-06A_1x06_P2.54mm_Vertical, symbol Connector:Conn_01x06_Pin
- 220in1: footprint TerminalBlock:TerminalBlock_Altech_AK300-3_P5.00mm -> TerminalBlock_Phoenix:TerminalBlock_Phoenix_MKDS-1,5-3-5.08_1x03_P5.08mm_Horizontal
- acin1: footprint TerminalBlock_MetzConnect:TerminalBlock_MetzConnect_Type011_RT05502HBWC_1x02_P5.00mm_Horizontal -> TerminalBlock_Phoenix:TerminalBlock_Phoenix_MKDS-1,5-2-5.08_1x02_P5.08mm_Horizontal
- r34, r35: value 3.3K -> 2.5K
Connections:
- net ADC_IN2 is gone; now on net MDO1: mcu1.15 (PA5)
- net AIN2 is gone; now on net AGND: AIN1.3 (Pin_3)
- net UART1_RX is gone; now on net MCU_RX: mcu1.31 (PA10)
- net UART1_TX is gone; now on net MCU_TX: mcu1.30 (PA9)
- net +5V: now also AIN1.1 (Pin_1)
- net AGND: no longer AIN1.2 (Pin_2)
- net AIN1: now also AIN1.2 (Pin_2); no longer AIN1.1 (Pin_1)
- net COM1: now also DDO1.8 (Pin_8); no longer DDO1.1 (Pin_1)
- net COM2: now also DDO1.6 (Pin_6); no longer DDO1.3 (Pin_3)
- net COM3: now also DDO1.3 (Pin_3); no longer DDO1.5 (Pin_5)
- net COM4: now also DDO1.1 (Pin_1); no longer DDO1.7 (Pin_7)
- net D220_IN1: now also mcu1.19 (PB1)
- net D220_IN2: now also mcu1.20 (PB2)
- net DI5: now also mcu1.45 (PB8)
- net DI6: now also mcu1.46 (PB9)
- net DO1: now also DDO1.7 (Pin_7); no longer DDO1.2 (Pin_2)
- net DO2: now also DDO1.5 (Pin_5); no longer DDO1.4 (Pin_4)
- net DO3: now also DDO1.4 (Pin_4); no longer DDO1.6 (Pin_6)
- net DO4: now also DDO1.2 (Pin_2); no longer DDO1.8 (Pin_8)
- net MDO2: now also mcu1.16 (PA6)
- net MDO3: now also mcu1.17 (PA7)
- net MDO4: now also mcu1.18 (PB0)
- net MGND: now also modout1.3 (Pin_3)
- net RELOUT11: now also relo1.2 (Pin_2)
- net RELOUT12: now also relo1.1 (Pin_1)
- net RELOUT21: now also relo1.4 (Pin_4)
- net RELOUT22: now also relo1.3 (Pin_3)
- net RS485_AO: now also modout1.2 (Pin_2)
- net RS485_BO: now also modout1.1 (Pin_1)
- net RS_SEL: now also mcu1.29 (PA8)
- net rlo1: now also mcu1.22 (PB11)
- net rlo2: now also mcu1.21 (PB10)
- net NOC renamed NOC1
- net NOC1: now also relo1.5 (Pin_5); no longer relay2.4
- new net NOC2: relay2.4, relo1.6 (Pin_6)
Other:
- moved on the sheet: 220in1
