File: test.kicad_sch (KiCad schematic)
At the start: 155 parts, among them Q1 T2N7002AK, Q2 T2N7002AK, SW1 SW_Push, U1 ESP32-S3-WROOM-1, U2 LD1117S33TR_SOT223, U3 SN75176AD, U4 LM321

Commit message: all done except gnds and vccs
Parts:
- removed PS1: HLK-5M05, Converter_ACDC:Converter_ACDC_Hi-Link_HLK-5Mxx, symbol Converter_ACDC:HLK-5M05
- added Ds1: SS34, Diode_SMD:D_SMA, symbol Diode:SS34
- added L24: L, Inductor_THT:L_Radial_D9.5mm_P5.00mm_Fastron_07HVP, symbol Device:L
- added PS1: HLK-5M24, Converter_ACDC:Converter_ACDC_Hi-Link_HLK-5Mxx, symbol Converter_ACDC:HLK-5M24
- added U5: LM2576HVS-5, Package_TO_SOT_SMD:TO-263-5_TabPin3, symbol Regulator_Switching:LM2576HVS-5
- added crs1, crs2: C_Polarized, Capacitor_THT:CP_Radial_D10.0mm_P3.80mm, symbol Device:C_Polarized
- cr2, cr3: footprint Capacitor_THT:CP_Radial_D22.0mm_P10.00mm_SnapIn -> Capacitor_THT:CP_Radial_D10.0mm_P3.80mm
Connections:
- net +5V: now also L24.1, U5.4 (FB), crs2.1; no longer dr1.1 (K), dr2.1 (K), pwrs1.2 (B), relay1.5, relay2.5
- net D05_IN5: now also mcu1.46 (PB9)
- net D05_IN6: now also mcu1.45 (PB8)
- net D24_IN1: now also mcu1.38 (PA15)
- net D24_IN2: now also mcu1.41 (PB5)
- net D24_IN3: now also mcu1.40 (PB4)
- net D24_IN4: now also mcu1.39 (PB3)
- net DI5: no longer mcu1.45 (PB8)
- net DI6: no longer mcu1.46 (PB9)
- net GND: now also Ds1.2 (A), PS1.3 (-Vout), U5.3 (GND), U5.5 (~{ON}/OFF), crs1.2, crs2.2
- net L: now also PS1.1 (AC/L)
- net N: now also PS1.2 (AC/N)
- net at pwrs1.1 (A): now also PS1.4 (+Vout)
- new net: Ds1.1 (K), L24.2, U5.2 (OUT)
- new net +24V: U5.1 (VIN), crs1.1, dr1.1 (K), dr2.1 (K), pwrs1.2 (B), relay1.5, relay2.5

Commit message: all done but gnd
Parts:
- removed SW1: SW_Push, Button_Switch_SMD:SW_Push_1P1T_NO_6x6mm_H9.5mm, symbol Switch:SW_Push
- added D1: LED, LED_SMD:LED_0805_2012Metric_Pad1.15x1.40mm_HandSolder, symbol Device:LED
- added U6: MAX31855KASA, Package_SO:SOIC-8_3.9x4.9mm_P1.27mm, symbol Sensor_Temperature:MAX31855KASA
- added cx1: 100nF, Capacitor_SMD:C_0805_2012Metric_Pad1.18x1.45mm_HandSolder, symbol Device:C
- added mcur1: Conn_01x02_Pin, Connector_PinHeader_2.54mm:PinHeader_1x02_P2.54mm_Vertical, symbol Connector:Conn_01x02_Pin
- added mxin1: Screw_Terminal_01x02, TerminalBlock_Phoenix:TerminalBlock_Phoenix_MKDS-1,5-2-5.08_1x02_P5.08mm_Horizontal, symbol Connector:Screw_Terminal_01x02
- added mxj1: 0, Resistor_SMD:R_0805_2012Metric_Pad1.20x1.40mm_HandSolder, symbol Device:R
- added rled1: 1K, Resistor_SMD:R_0805_2012Metric_Pad1.20x1.40mm_HandSolder, symbol Device:R_US
Connections:
- net 3.3V is gone; now on net +3.3V: espio1.21 (Pin_21)
- net +3.3V: now also U6.4 (V_CC), cx1.1
- net GND: now also D1.1 (K), U6.1 (GND), cx1.2, mcur1.2 (Pin_2), mxj1.1
- net RELOUT11: now also relo1.4 (Pin_4); no longer relo1.2 (Pin_2)
- net RELOUT12: now also relo1.3 (Pin_3); no longer relo1.1 (Pin_1)
- net RELOUT21: now also relo1.2 (Pin_2); no longer relo1.4 (Pin_4)
- net RELOUT22: now also relo1.1 (Pin_1); no longer relo1.3 (Pin_3)
- net RESET: now also mcur1.1 (Pin_1)
- net SCK: now also U6.5 (SCK)
- net SO: now also U6.7 (SO)
- net MXCS: now reaches mcu1.32 (PA11)
- net MXCS: now also U6.6 (~{CS})
- net LED: now reaches mcu1.4 (PC15)
- net LED: now also rled1.1
- new net: D1.2 (A), rled1.2
- new net: U6.2 (T-), mxin1.1 (Pin_1), mxj1.2
- new net: U6.3 (T+), mxin1.2 (Pin_2)
